File: KiCAD/PC8001-MEM.kicad_pcb (KiCad board)
At the start: 2 copper layers, 100 x 75 mm, 33 parts, among them J1 PC-8001 ext BUS, U1 74LS32, U10 628128, U2 74LS138, U3 ULN2003A, U4 74LS138, U5 74LS175, U6 74LS32, U7 74LS541, U8 74LS273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

Commit message: 8k SRAMボードコントロール信号端子追加・ガーバーデータ再出力
Parts:
- added J2: MEM-CON, Connector_PinHeader_2.54mm:PinHeader_1x02_P2.54mm_Vertical, F.Cu at (99.0, 68.5)
Connections:
- J1 pad 14: /~INT -> (no net)
- J1 pad 16: /~NMI -> (no net)
- J1 pad 18: /~EXTON -> (no net)
- J1 pad 2: /+12V -> (no net)
- J1 pad 38: /~WAIT -> (no net)
- J1 pad 4: /-12V -> (no net)
- J1 pad 40: /~WE -> (no net)
- J1 pad 42: /~MUX -> (no net)
- J1 pad 43: /~RFSH -> (no net)
- J1 pad 44: /~RAS0 -> (no net)
- J1 pad 45: /~M1 -> (no net)
- J1 pad 46: /~RAS1 -> (no net)
- J1 pad 47: /SCLOCK -> (no net)
- J1 pad 49: /CLK -> (no net)
- U10 pad 1: Net-(U10-Pad1) -> (no net)
- U2 pad 10: Net-(U2-Pad10) -> (no net)
- U2 pad 11: Net-(U2-Pad11) -> (no net)
- U2 pad 12: Net-(U2-Pad12) -> (no net)
- U2 pad 13: Net-(U2-Pad13) -> (no net)
- U2 pad 14: Net-(U2-Pad14) -> (no net)
- U2 pad 15: Net-(U2-Pad15) -> (no net)
- U2 pad 9: Net-(U2-Pad9) -> (no net)
- U3 pad 10: Net-(U3-Pad10) -> (no net)
- U3 pad 11: Net-(U3-Pad11) -> (no net)
- U3 pad 12: Net-(U3-Pad12) -> (no net)
- U3 pad 9: Net-(U3-Pad9) -> (no net)
- U4 pad 14: Net-(U4-Pad14) -> (no net)
- U4 pad 15: Net-(U4-Pad15) -> (no net)
- U4 pad 7: Net-(U4-Pad7) -> (no net)
- U4 pad 9: Net-(U4-Pad9) -> (no net)
- U5 pad 10: Net-(U5-Pad10) -> (no net)
- U5 pad 11: Net-(U5-Pad11) -> (no net)
- U5 pad 14: Net-(U5-Pad14) -> (no net)
- U5 pad 15: Net-(U5-Pad15) -> (no net)
- U6 pad 11: Net-(U6-Pad11) -> (no net)
- U6 pad 8: Net-(U6-Pad8) -> (no net)
Routing:
- net /E2-D4: track 104.8 -> 117.7 mm
- net /E2-D0: track 92.5 -> 101.5 mm, vias 0 -> 1
Other:
- board text added: "KUNI-NET 2021"
- board text added: "PC-8001 128kB Memory Board [KP80-MEM128]"
- board text removed: "KUNI-NET 2020"
- board text removed: "PC-8001 128kB Memory Board <KP80-MEM128>"
